File: Week11/Joseto/Step.sch (EAGLE design)
At the start: 5 parts, among them IC1 ATTINY44-SSU

Commit message: la cague
Parts:
- added U$3: PINHD-2X2-SMD, fab:PINHD-2X2-SMD
Changed lines of the file:
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@@
 <part name="P+5" library="supply1" library_urn="urn:adsk.eagle:library:371" deviceset="VCC" device=""/>
 <part name="C1" library="fab" deviceset="CAP-US" device="1206FAB" value="1uF"/>
+<part name="U$3" library="fab" deviceset="PINHD-2X2-SMD" device=""/>
 </parts>
 <sheets>
@@
 <attribute name="VALUE" x="182.6" y="75.39" size="1.778" layer="96" rot="R270"/>
 </instance>
+<instance part="U$3" gate="G$1" x="62.2" y="24.2" smashed="yes">
+<attribute name="NAME" x="53.31" y="29.915" size="1.778" layer="95"/>
+<attribute name="VALUE" x="53.31" y="19.12" size="1.778" layer="96"/>
+</instance>
 </instances>
