File: Final Project/Ultrasonic/ArduinoBase.brd (EAGLE design)
At the start: 33.7 x 31.4 mm, 19 parts, among them IC1 ATTINY44-SSU, IC3 OPAMPSOT23-5

Commit message: Sensor ultrasonico
Parts:
- R4, R5: value 10K -> 10
- R6: value 10K -> 0
Changed lines of the file:
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@@
 <attribute name="VALUE" x="12.446" y="21.59" size="1.016" layer="27" ratio="15" rot="R180"/>
 </element>
-<element name="R4" library="fab" package="R1206FAB" value="10K" x="6.858" y="18.542" smashed="yes" rot="R270">
+<element name="R4" library="fab" package="R1206FAB" value="10" x="6.858" y="18.542" smashed="yes" rot="R270">
 <attribute name="NAME" x="8.128" y="20.32" size="1.016" layer="25" ratio="15" rot="R270"/>
 <attribute name="VALUE" x="4.572" y="20.32" size="1.016" layer="27" ratio="15" rot="R270"/>
 </element>
-<element name="R5" library="fab" package="R1206FAB" value="10K" x="17.78" y="20.828" smashed="yes">
+<element name="R5" library="fab" package="R1206FAB" value="10" x="17.78" y="20.828" smashed="yes">
 <attribute name="NAME" x="16.002" y="22.098" size="1.016" layer="25" ratio="15"/>
 <attribute name="VALUE" x="16.002" y="18.542" size="1.016" layer="27" ratio="15"/>
@@
 <attribute name="VALUE" x="-0.254" y="9.398" size="1.27" layer="21" rot="R270"/>
 </element>
-<element name="R6" library="fab" package="R1206FAB" value="10K" x="11.7856" y="10.8458" smashed="yes" rot="R90">
+<element name="R6" library="fab" package="R1206FAB" value="0" x="11.7856" y="10.8458" smashed="yes" rot="R90">
 <attribute name="NAME" x="10.5156" y="9.0678" size="1.016" layer="25" ratio="15" rot="R90"/>
 <attribute name="VALUE" x="14.0716" y="9.0678" size="1.016" layer="27" ratio="15" rot="R90"/>
