File: Final Project/Ultrasonic/ArduinoBase.sch (EAGLE design)
At the start: 8 parts, among them IC1 ATTINY44-SSU

Commit message: Sensor
Parts:
- added D1: (no value), fab:DIODESOD123
- added GND, U$5, U$6: PINHD-2X2-SMD, fab:PINHD-2X2-SMD
- added IC2: (no value), fab:REGULATORSOT23
- added IC3: OPAMPSOT23-5, fab:OPAMPSOT23-5
- added R3, R4, R5, R6, R7: 10K, fab:RES-US1206FAB
Connections:
- removed net N$2: R1.1
- removed net TX: IC1.(PCINT0/AREF/ADC0)PA0, U$1.TXD
- new net 12V: GND.1, GND.2, IC2.IN, IC3.V-, R6.1, R6.2
- new net ANALOG: IC3.OUT, R5.1
- new net N$11: IC3.-IN, R3.1, R4.2
- new net N$3: IC3.+IN, R5.2, R7.1
- new net N$9: D1.C, IC2.OUT
- new net PWM: IC1.(PCINT7/ICP/OC0B/ADC7)PA7, U$5.1, U$5.2
- new net TRANS1: R7.2, U$6.1, U$6.2
- new net TRANS2: R3.2, U$6.3, U$6.4
- net 0: now also GND.3, GND.4, IC2.GND, IC3.V+, R1.1, R4.1, U$5.3, U$5.4
- net MISO: no longer IC1.(PCINT7/ICP/OC0B/ADC7)PA7
- net VCC: now also D1.A

Commit message: Sensor ultrasonico
Parts:
- R4, R5: value 10K -> 10
- R6: value 10K -> 0
Changed lines of the file:
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@@
 <part name="U$6" library="fab" deviceset="PINHD-2X2-SMD" device=""/>
 <part name="R3" library="fab" deviceset="RES-US" device="1206FAB" value="10K"/>
-<part name="R4" library="fab" deviceset="RES-US" device="1206FAB" value="10K"/>
-<part name="R5" library="fab" deviceset="RES-US" device="1206FAB" value="10K"/>
-<part name="R6" library="fab" deviceset="RES-US" device="1206FAB" value="10K"/>
+<part name="R4" library="fab" deviceset="RES-US" device="1206FAB" value="10"/>
+<part name="R5" library="fab" deviceset="RES-US" device="1206FAB" value="10"/>
+<part name="R6" library="fab" deviceset="RES-US" device="1206FAB" value="0"/>
 <part name="R7" library="fab" deviceset="RES-US" device="1206FAB" value="10K"/>
 </parts>
