File: Final Project/Ultrasonic/Board/Ultrasonic.brd (EAGLE design)
At the start: 100 x 80 mm, 17 parts, among them IC1 ATTINY44-SSU, IC3 OPAMPSOT23-5

Commit message: Ultrasonic Fail :(
Parts:
- R3, R7: value 10K -> 100k
- R4, R5: value 10 -> 1k
Changed lines of the file:
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@@
 <attribute name="VALUE" x="19.177" y="10.6934" size="1.016" layer="27" ratio="15" rot="R270"/>
 </element>
-<element name="R3" library="fab" package="R1206FAB" value="10K" x="2.4638" y="27.5336" smashed="yes" rot="R90">
+<element name="R3" library="fab" package="R1206FAB" value="100k" x="2.4638" y="27.5336" smashed="yes" rot="R90">
 <attribute name="NAME" x="1.1938" y="25.7556" size="1.016" layer="25" ratio="15" rot="R90"/>
 <attribute name="VALUE" x="4.7498" y="25.7556" size="1.016" layer="27" ratio="15" rot="R90"/>
 </element>
-<element name="R4" library="fab" package="R1206FAB" value="10" x="2.2352" y="22.1488" smashed="yes" rot="R90">
+<element name="R4" library="fab" package="R1206FAB" value="1k" x="2.2352" y="22.1488" smashed="yes" rot="R90">
 <attribute name="NAME" x="0.9652" y="20.3708" size="1.016" layer="25" ratio="15" rot="R90"/>
 <attribute name="VALUE" x="4.5212" y="20.3708" size="1.016" layer="27" ratio="15" rot="R90"/>
 </element>
-<element name="R5" library="fab" package="R1206FAB" value="10" x="10.0584" y="19.8882" smashed="yes" rot="R90">
+<element name="R5" library="fab" package="R1206FAB" value="1k" x="10.0584" y="19.8882" smashed="yes" rot="R90">
 <attribute name="NAME" x="8.7884" y="18.1102" size="1.016" layer="25" ratio="15" rot="R90"/>
 <attribute name="VALUE" x="12.3444" y="18.1102" size="1.016" layer="27" ratio="15" rot="R90"/>
 </element>
-<element name="R7" library="fab" package="R1206FAB" value="10K" x="8.3312" y="25.8826" smashed="yes" rot="R180">
+<element name="R7" library="fab" package="R1206FAB" value="100k" x="8.3312" y="25.8826" smashed="yes" rot="R180">
 <attribute name="NAME" x="10.1092" y="24.6126" size="1.016" layer="25" ratio="15" rot="R180"/>
 <attribute name="VALUE" x="10.1092" y="28.1686" size="1.016" layer="27" ratio="15" rot="R180"/>
