File: Final Project/PlacaMotor/Mosfet2.sch (EAGLE design)
At the start: 7 parts, among them IC1 ATTINY44-SSU

Commit message: Placa Motor
Parts:
- removed U$1: FTDI-SMD-HEADER, fab:FTDI-SMD-HEADER
- added D1: (no value), fab:DIODESOD123
- added IC2: (no value), fab:REGULATORSOT23
- added R3, R4: 0, fab:RES-US1206FAB
- added T2: (no value), fab:NMOSFETTO252
- added U$4, U$5: PINHD-2X2-SMD, fab:PINHD-2X2-SMD
- added VR1: 5k, SparkFun-Resistors:TRIMPOT-SMD-5MM-CLOSED-1/4W-20%
Connections:
- removed net N$13: IC1.(PCINT2/AIN1/ADC2)PA2
- new net 12V: IC2.IN, U$4.1, U$4.2, U$5.1, U$5.2
- new net ANALOG: IC1.(PCINT2/AIN1/ADC2)PA2, VR1.WIPER
- new net MOSFET: T2.D, U$5.3, U$5.4
- new net MOTOR: IC1.(PCINT7/ICP/OC0B/ADC7)PA7, T2.G
- new net N$11: D1.C, IC2.OUT
- net 0: now also IC2.GND, T2.S, U$4.3, U$4.4, VR1.CW; no longer U$1.GND
- net MISO: no longer IC1.(PCINT7/ICP/OC0B/ADC7)PA7
- net RX: no longer U$1.RXD
- net TX: no longer U$1.TXD
- net VCC: now also D1.A, R3.1, R3.2, R4.1, R4.2, VR1.CCW; no longer U$1.VCC
Other:
- note removed: "SERIAL/FTDI"
