File: Final Project/PlacaMotor/MosfetV3.brd (EAGLE design)
At the start: 36.3 x 37.5 mm, 14 parts, among them IC1 ATTINY44-SSU

Commit message: Placa FTDI
Parts:
- added U$1: FTDI-SMD-HEADER, fab:1X06SMD
- moved IC1 6.15 mm to (18.8, 11.3)
- moved R2 6.15 mm to (24.3, 9.40)
- moved T2 6.15 mm to (31.5, 30.4)
- moved U$3 6.15 mm to (18.8, 27.8)
- moved U$5 6.15 mm to (33.0, 4.34)
- moved C1 6.15 mm to (12.5, 30.4)
- moved U$2 6.15 mm to (21.4, 21.5)
- moved D1 6.15 mm to (29.8, 11.9)
- moved IC2 6.15 mm to (26.6, 16.0)
- moved R1 6.15 mm to (9.96, 20.2)
- moved R3 6.15 mm to (16.4, 5.21)
- moved R4 6.15 mm to (28.2, 7.65)
- moved U$4 6.15 mm to (32.8, 20.2)
- moved VR1 6.15 mm to (9.96, 8.79)
Connections:
- net 0: now also U$1.1
- net RX: now also U$1.5
- net TX: now also U$1.4
- net VCC: now also U$1.3
Routing:
- net VCC: track 62.6 -> 79.0 mm
- net 0: track 98.8 -> 114.4 mm
- net RX: track 0.00 -> 13.3 mm
- net TX: track 0.00 -> 12.1 mm
Other:
- board size 36.3 x 37.5 mm -> 42.2 x 37.3 mm

Commit message: Codigos G
Other:
- board size 42.2 x 37.3 mm -> 42.1 x 37.4 mm
Changed lines of the file:
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@@
 <plain>
 <wire x1="0.381" y1="-0.1524" x2="42.4436" y2="-0.2032" width="0" layer="20"/>
-<wire x1="42.4436" y1="-0.2032" x2="42.342" y2="37.0486" width="0" layer="20"/>
-<wire x1="42.342" y1="37.0486" x2="0.2794" y2="37.0994" width="0" layer="20"/>
-<wire x1="0.2794" y1="37.0994" x2="0.381" y2="-0.1524" width="0" layer="20"/>
+<wire x1="42.4436" y1="-0.2032" x2="42.4436" y2="37.1502" width="0" layer="20"/>
+<wire x1="42.4436" y1="37.1502" x2="0.381" y2="37.201" width="0" layer="20"/>
+<wire x1="0.381" y1="37.201" x2="0.381" y2="-0.1524" width="0" layer="20"/>
 </plain>
 <attributes>
