File: Final Project/PlacaMotor/MosfetV5.brd (EAGLE design)
At the start: 55.9 x 39.6 mm, 23 parts, among them IC1 ATTINY44-SSU

Commit message: lala
Changed lines of the file:
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@@
 <contactref element="U$7" pad="1"/>
 <wire x1="31.1366" y1="6.5024" x2="31.1366" y2="8.41866875" width="0.4" layer="1"/>
-<wire x1="31.1366" y1="8.41866875" x2="31.6388" y2="8.92086875" width="0.4" layer="1"/>
-<wire x1="31.6388" y1="8.92086875" x2="31.6388" y2="12.0904" width="0.4" layer="1"/>
-<wire x1="31.6388" y1="12.0904" x2="35.0647" y2="12.0904" width="0.4" layer="1"/>
 <wire x1="35.0647" y1="12.0904" x2="35.1409" y2="12.0142" width="0.4" layer="1"/>
+<wire x1="31.77033125" y1="9.0524" x2="32.258" y2="9.0524" width="0.4" layer="1"/>
+<wire x1="32.258" y1="9.0524" x2="32.3088" y2="9.1032" width="0.4" layer="1"/>
+<wire x1="32.3088" y1="9.1032" x2="32.3088" y2="11.9888" width="0.4" layer="1"/>
+<wire x1="32.3088" y1="11.9888" x2="32.3342" y2="12.0142" width="0.4" layer="1"/>
+<wire x1="32.3342" y1="12.0142" x2="35.1409" y2="12.0142" width="0.4" layer="1"/>
+<wire x1="31.1366" y1="8.41866875" x2="31.77033125" y2="9.0524" width="0.4" layer="1"/>
 </signal>
 <signal name="CRYSTAL2">
@@
 <contactref element="R4" pad="1"/>
 <contactref element="IC1" pad="11"/>
-<wire x1="29.9339" y1="13.2842" x2="19.8405" y2="13.2842" width="0.4" layer="1"/>
-<wire x1="19.8405" y1="13.2842" x2="19.8405" y2="14.5446" width="0.4" layer="1"/>
-<wire x1="9.4488" y1="17.8338" x2="9.4488" y2="19.685" width="0.4" layer="1"/>
-<wire x1="15.9289" y1="16.4496" x2="11.0013" y2="16.4496" width="0.4" layer="1"/>
-<wire x1="11.0013" y1="16.4496" x2="11.0013" y2="17.8338" width="0.4" layer="1"/>
-<wire x1="11.0013" y1="17.8338" x2="9.4488" y2="17.8338" width="0.4" layer="1"/>
-<wire x1="15.9289" y1="14.5446" x2="15.9289" y2="16.4496" width="0.4" layer="1"/>
-<wire x1="19.8405" y1="14.5446" x2="15.9289" y2="14.5446" width="0.4" layer="1"/>
+<wire x1="19.8405" y1="13.2842" x2="29.9339" y2="13.2842" width="0.4" layer="1"/>
 <wire x1="9.4488" y1="19.685" x2="9.4488" y2="23.3022" width="0.4" layer="1"/>
 <wire x1="9.4488" y1="23.3022" x2="9.4888" y2="23.3022" width="0.4" layer="1"/>
+<wire x1="9.4488" y1="19.685" x2="9.525" y2="19.6088" width="0.4" layer="1"/>
+<wire x1="9.525" y1="19.6088" x2="9.525" y2="18.2372" width="0.4" layer="1"/>
+<wire x1="9.525" y1="18.2372" x2="9.779" y2="17.9832" width="0.4" layer="1"/>
+<wire x1="11.8364" y1="17.9832" x2="11.8364" y2="16.9164" width="0.4" layer="1"/>
+<wire x1="11.8364" y1="16.9164" x2="16.383" y2="16.9164" width="0.4" layer="1"/>
+<wire x1="9.779" y1="17.9832" x2="11.8364" y2="17.9832" width="0.4" layer="1"/>
+<wire x1="16.383" y1="16.9164" x2="16.383" y2="15.0368" width="0.4" layer="1"/>
+<wire x1="16.383" y1="15.0368" x2="19.8405" y2="15.0368" width="0.4" layer="1"/>
+<wire x1="19.8405" y1="15.0368" x2="19.8405" y2="13.2842" width="0.4" layer="1"/>
 </signal>
 <signal name="ENC1">
